File: hardware/RPN_Scientific_Calculator.kicad_sch (KiCad schematic)
At the start: 80 parts, among them J1 PICKIT4/5, Q1 2N7002H, Q2 AO3415A, SW1 x*y/(x+y), SW10 x↔y/last x, SW11 8, SW12 5, SW13 2, SW14 ./e, SW15 f1/modes, SW16 x^{y}/x√y, SW17 sin/sin^{-1}, SW18 9, SW19 6, SW2 √x/3√x, SW20 3, SW21 E/π, SW22 f2/disp, SW23 log/10^{x}, SW24 cos/cos^{-1}, SW25 +/-, SW26 ×/x!, SW27 +, SW28 Shift, SW29 POWER, SW3 R↓, SW30 f3, SW31 ln/e^{x}, SW32 tan/tan^{-1}, SW33 ←/OFF, SW34 ÷/x^{-1}, SW35 -, SW36 Enter, SW4 7, SW5 4, SW6 1, SW7 0, SW8 f_{c}RC/f_{c}LC, SW9 x^{2}/x^{3}, U1 AQM1602Y-RN-GBW, U2 XC9140, U3 PIC32CM5164LE00048

Commit message: 回路図の修正
Parts:
- R1, R2: value 4.7k -> 10k
- R10, R11, R7, R8, R9: now fitted
Changed lines of the file:
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@@
 		(in_bom yes)
 		(on_board yes)
-		(dnp yes)
+		(dnp no)
 		(fields_autoplaced yes)
 		(property "Reference" "R9"
@@
 		(in_bom yes)
 		(on_board yes)
-		(dnp yes)
+		(dnp no)
 		(fields_autoplaced yes)
 		(property "Reference" "R10"
@@
 		(in_bom yes)
 		(on_board yes)
-		(dnp yes)
+		(dnp no)
 		(fields_autoplaced yes)
 		(property "Reference" "R8"
@@
 			)
 		)
-		(property "Value" "4.7k"
+		(property "Value" "10k"
 			(at 40.64 115.5699 0)
 			(effects
@@
 			)
 		)
-		(property "Value" "4.7k"
+		(property "Value" "10k"
 			(at 31.75 115.5699 0)
 			(effects
@@
 		(in_bom yes)
 		(on_board yes)
-		(dnp yes)
+		(dnp no)
 		(fields_autoplaced yes)
 		(property "Reference" "R11"
@@
 		(in_bom yes)
 		(on_board yes)
-		(dnp yes)
+		(dnp no)
 		(fields_autoplaced yes)
 		(property "Reference" "R7"
